File: capstone_core/power_system.kicad_sch (KiCad schematic)
At the start: 26 parts, among them U1 LM2596S-12, U2 LM2596S-12, U3 LP2985-3.3

Commit message: up to date project
Parts:
- removed U2: LM2596S-12, Package_TO_SOT_SMD:TO-263-5_TabPin3, symbol Regulator_Switching:LM2596S-12
- gave numbers to parts that had none: 4
- renumbered C2 to C1, C7 to C10, C4 to C11, C8 to C12, C5 to C2, C9 to C3, C1 to C4, C6 to C5, C10 to C6, C11 to C7, C3 to C9, R3 to R2, R2 to R3, U3 to U1, U1 to U2
Connections:
- net +12V_RAW renamed +V_BATT
- net +12V_REG renamed +12V
